File: Atlantis_board/ClusterMonitor_2floor_atlantisModule_moscow.kicad_pcb (KiCad board)
At the start: 2 copper layers, 400 x 159.3 mm, 185 parts, among them J1 RJ45_Molex_smd_44144-0003, J2 Conn_01x07, SW1 SW_SPST_Double, SW2 ADDRESS_SELECT, SW3 SW_SPDT, U1 AMS1117-3.3, U2 STM32F030C8Tx

Commit message: Some changes
Add stencil board layout.
Add gerbers.
Minor changes in expancion and atrium board.
Parts:
- moved R5 5.92 mm to (-97.8, -14.2)
- moved D4 5.92 mm to (-97.6, -15.7), turned to 0 degrees
- moved C2 0.51 mm to (-147.6, -5.84)
- moved D1 0.21 mm to (-142.1, 4.24)
Routing:
- net +5V: track 379.3 -> 394.2 mm
- net SWITCH_MODE: track 17.4 -> 11.3 mm
- net VDDA: track 179.3 -> 182.6 mm
- net Net-(R5-Pad2): track 10.2 -> 7.24 mm
- net GND: track 213.6 -> 214.8 mm
