File: Expansion_board/Cluster_LED_monitor.kicad_pcb (KiCad board)
At the start: 2 copper layers, 267.5 x 85 mm, 37 parts, among them J1 Raspberry_Pi_2_3, J10 RJ45, J11 Conn_01x02, J2 Conn_01x02_Female, J3 RJ45, J4 RJ45, J5 RJ45, J6 RJ45, J7 RJ45, J8 RJ45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

Commit message: Some changes
Add stencil board layout.
Add gerbers.
Minor changes in expancion and atrium board.
Parts:
- moved G*** 5.92 mm to (173.0, 120.7)
- moved G*** 5.87 mm to (130.8, 98.8)
- moved C1 4.87 mm to (57.2, 101.6), turned to 0 degrees
- moved R6 4.62 mm to (62.0, 104.4)
- moved J10 0.17 mm to (75.0, 63.0)
- moved J8 0.17 mm to (127.0, 63.0)
- moved J9 0.17 mm to (101.0, 63.0)
- renumbered J6 to J4, J9 to J6, J8 to J7, J4 to J8, J7 to J9
Routing:
- net +5V: track 86.5 -> 229.9 mm, vias 11 -> 14
- net GND: track 72.2 -> 112.3 mm, vias 20 -> 47
- net I2C_SDA: track 381.7 -> 395.2 mm
- net I2C_SCL: track 402.1 -> 410.9 mm
- net Net-(J11-Pad1): track 180.3 -> 173.5 mm
- net Net-(J1-Pad7): track 131.8 -> 125.1 mm
- net Net-(R1-Pad2): track 75.2 -> 76.9 mm, vias 0 -> 2
- net Net-(R3-Pad2): vias 0 -> 2
Other:
- board text added: "M2.5"
- board text added: "M3"
- board text added: "Raspberry Pi Zero W"
