File: Mirage_board/ClusterMonitor_2floor_mirageModule_moscow.kicad_pcb (KiCad board)
At the start: 2 copper layers, 132.8 x 325.5 mm, 199 parts, among them J1 RJ45_Molex_smd_44144-0003, J2 Conn_01x07, SW1 SW_SPST_Double, SW2 ADDRESS_SELECT, SW3 SW_SPDT, U1 AMS1117-3.3, U2 STM32F030C8Tx

Commit message: Some changes
Add stencil board layout.
Add gerbers.
Minor changes in expancion and atrium board.
Parts:
- moved G*** 60.6 mm to (-73.0, 97.2)
- moved D4 5.85 mm to (-131.2, 11.5), turned to 270 degrees
- moved R5 5.85 mm to (-132.7, 11.3)
- moved C2 2.13 mm to (-155.4, 53.8), turned to 270 degrees
Routing:
- net +5V: track 224.4 -> 245.4 mm
- net GND: track 71.0 -> 63.7 mm, vias 33 -> 30
- net SWITCH_MODE: track 17.3 -> 11.9 mm
- net Net-(R5-Pad2): track 10.2 -> 6.59 mm
- net VDDA: track 196.2 -> 199.3 mm
