File: Oasis_board/ClusterMonitor_2floor_oasisModule_moscow.kicad_pcb (KiCad board)
At the start: 2 copper layers, 132.8 x 325.1 mm, 149 parts, among them J1 RJ45_Molex_smd_44144-0003, J2 Conn_01x07, SW1 SW_SPST_Double, SW2 ADDRESS_SELECT, SW3 SW_SPDT, U1 AMS1117-3.3, U2 STM32F030C8Tx

Commit message: Some changes
Add stencil board layout.
Add gerbers.
Minor changes in expancion and atrium board.
Parts:
- moved D4 10.5 mm to (-146.6, 103.5), turned to 90 degrees
- moved R5 10.5 mm to (-145.0, 103.8)
- moved D2 10.4 mm to (-139.1, 135.1)
- moved R2 10.4 mm to (-137.2, 135.1)
- moved TEST2 10.4 mm to (-139.1, 137.7)
- moved D1 7.12 mm to (-146.2, 135.1)
- moved R1 7.12 mm to (-144.3, 135.1)
- moved TEST1 7.12 mm to (-146.2, 137.7)
- moved TEST3 4.27 mm to (-142.4, 141.0)
- moved C2 1.17 mm to (-139.3, 157.4)
Routing:
- net +5V: track 182.6 -> 192.3 mm
- net VDDA: track 171.2 -> 178.5 mm
- net Net-(R5-Pad2): track 10.2 -> 4.55 mm
- net GND: track 119.2 -> 116.6 mm, vias 32 -> 33
- net SWITCH_MODE: track 16.4 -> 15.8 mm
