File: Atrium_Central_board/ClusterMonitor_2floor_atriumModule_moscow_ricky_version.kicad_pcb (KiCad board)
At the start: 2 copper layers, 135.1 x 143.6 mm, 52 parts, among them J1 RJ32_Shielded, J2 Conn_01x07, SW1 SW_SPST, SW2 ADDRESS_SELECT, SW3 SW_SPDT, U1 AMS1117-3.3, U2 STM32F030C8Tx

Commit message: Atrium pcb bomanyte version
Parts:
- added G***: LOGO, ClusterMonitor_silklib:label_atrium_silk_kicad, B.Cu at (264.2, 43.8)
- C10: value 4.7uF -> CP_EIA-3216-10_Kemet-I_Pad1.58x1.35mm_HandSolder
- moved R4 52.6 mm to (249.7, 89.6)
- moved D3 49.4 mm to (249.7, 87.9), turned to 0 degrees
- moved 3v3 20.4 mm to (206.5, 93.7)
- moved GND 10.2 mm to (227.2, 132.4)
- moved 5V 9.50 mm to (222.6, 132.5)
- moved C4 6.18 mm to (213.8, 84.0)
- moved D4 5.46 mm to (199.4, 69.8), turned to 0 degrees
- moved C10 4.91 mm to (211.6, 84.8), turned to 270 degrees
- moved C2 4.77 mm to (195.7, 80.2), turned to 90 degrees
- moved I2C1_SDA 3.73 mm to (216.4, 109.1)
- moved R5 3.45 mm to (200.2, 67.9), turned to 0 degrees
- moved R2 2.90 mm to (206.6, 91.1), turned to 180 degrees
- moved R1 2.23 mm to (222.6, 129.8)
- moved C5 1.30 mm to (208.7, 84.9)
- moved D2 1.20 mm to (206.5, 89.5), turned to 180 degrees
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- renumbered 3V3 to 3v3, 5V1 to 5V, GND1 to GND, I2C_SCL1 to I2C1_SCL, I2C_SDA1 to I2C1_SDA, SPI_CLK1 to SPI1_CLK, SPI_MOSI1 to SPI1_MOSI
Routing:
- net Net-(R4-Pad1): track 5.70 -> 65.1 mm
- net GND: track 115.6 -> 63.2 mm, vias 21 -> 27
- net +5V: track 69.8 -> 33.3 mm
- net SYS_JTMS-SWDIO: track 61.6 -> 44.8 mm
- net SWITCH_MODE: track 16.3 -> 20.6 mm
- net Net-(D1-Pad1): track 4.08 -> 1.93 mm
- net VDDA: track 127.8 -> 125.7 mm, vias 0 -> 1
- net REG_4b: track 18.8 -> 17.6 mm
- net SPI1_MOSI: track 71.5 -> 70.6 mm
- net C_RST: track 45.7 -> 44.8 mm
- net I2C1_SDA: track 64.3 -> 63.6 mm
- net REG_1b: track 19.3 -> 18.8 mm
Other:
- rule trace_min: 0.2 -> 0.127
- rule via_min_drill: 0.3 -> 0.2
- board text added: "JLCJLCJLCJLC"
- board text added: "RESET"
- board text added: "TEST_MODE"
- board text removed: "GND"
- board text removed: "RST"
- board text removed: "RX"
- board text removed: "SWCLK"
- board text removed: "SWDIO"
- board text removed: "TX"
- board text removed: "VDDA"
