File: Atrium_Central_board/ClusterMonitor_2floor_atriumModule_moscow.kicad_pcb (KiCad board)
At the start: 2 copper layers, 135.1 x 143.6 mm, 52 parts, among them J1 RJ32_Shielded, J2 Conn_01x07, SW1 SW_SPST, SW2 ADDRESS_SELECT, SW3 SW_SPDT, U1 AMS1117-3.3, U2 STM32F030C8Tx

Commit message: Atrium pcb tweaking
Parts:
- moved C10 4.82 mm to (212.3, 84.6), turned to 270 degrees
- moved R2 1.22 mm to (208.0, 89.9)
- moved C5 0.76 mm to (209.6, 85.0)
- moved C4 0.48 mm to (207.6, 84.1)
Routing:
- net +5V: track 69.8 -> 73.3 mm
- net GND: track 115.6 -> 118.4 mm
- net VDDA: track 127.8 -> 125.0 mm

Commit message: Add STM32 firmware
Parts:
- added G***: LOGO, ClusterMonitor_silklib:label_atrium_silk_kicad, B.Cu at (264.2, 58.2)
- renumbered 5V1 to 5V, GND1 to GND, I2C_SCL1 to I2C_SCL, I2C_SDA1 to I2C_SDA, SPI_CLK1 to SPI_CLK, SPI_MOSI1 to SPI_MOSI
Other:
- board text added: "3v3"
- board text added: "JLCJLCJLCJLC"
- board text removed: "VDDA"
